File: mpht_mcu.kicad_sch (KiCad schematic)
At the start: 11 parts, among them SW101 KMR421GULCLFS, SW102 KMR421GULCLFS, U1 ESP32-S3-WROOM-1-N4R2

Commit message: Added On/Off Switch Mode Selection Added a List of ToDos
Connections:
- net SLEEP_CTRL_PIN: now reaches U1.10 (IO17)
Other:
- moved on the sheet: D104, R115
Changed lines of the file:
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@@
 	(wire
 		(pts
-			(xy 199.39 60.96) (xy 199.39 63.5)
+			(xy 209.55 60.96) (xy 209.55 63.5)
 		)
 		(stroke
@@
 	(wire
 		(pts
-			(xy 199.39 68.58) (xy 199.39 69.85)
+			(xy 209.55 68.58) (xy 209.55 69.85)
 		)
 		(stroke
@@
 	(wire
 		(pts
-			(xy 199.39 74.93) (xy 199.39 78.74)
+			(xy 209.55 74.93) (xy 209.55 78.74)
 		)
 		(stroke
@@
 	(wire
 		(pts
+			(xy 176.53 68.58) (xy 187.96 68.58)
+		)
+		(stroke
+			(width 0)
+			(type default)
+		)
+	)
+	(wire
+		(pts
 			(xy 88.9 90.17) (xy 88.9 86.36)
 		)
@@
 	(wire
 		(pts
-			(xy 176.53 78.74) (xy 199.39 78.74)
+			(xy 176.53 78.74) (xy 209.55 78.74)
 		)
 		(stroke
@@
 		)
 	)
+	(hierarchical_label "SLEEP_CTRL_PIN"
+		(shape input)
+		(at 187.96 68.58 0)
+		(effects
+			(font
+				(size 1.27 1.27)
+			)
+			(justify left)
+		)
+	)
 	(hierarchical_label "CHRG_STAT1"
 		(shape input)
@@
 	(symbol
 		(lib_id "power:+3V3")
-		(at 199.39 60.96 0)
+		(at 209.55 60.96 0)
 		(unit 1)
 		(body_style 1)
@@
 		(fields_autoplaced yes)
 		(property "Reference" "#PWR0141"
-			(at 199.39 64.77 0)
+			(at 209.55 64.77 0)
 			(hide yes)
 			(show_name no)
@@
 		)
 		(property "Value" "+3V3"
-			(at 199.39 56.8269 0)
+			(at 209.55 56.8269 0)
 			(show_name no)
 			(do_not_autoplace no)
@@
 		)
 		(property "Footprint" ""
-			(at 199.39 60.96 0)
+			(at 209.55 60.96 0)
 			(hide yes)
 			(show_name no)
@@
 		)
 		(property "Datasheet" ""
-			(at 199.39 60.96 0)
+			(at 209.55 60.96 0)
 			(hide yes)
 			(show_name no)
@@
 		)
 		(property "Description" "Power symbol creates a global label with name \"+3V3\""
-			(at 199.39 60.96 0)
+			(at 209.55 60.96 0)
 			(hide yes)
 			(show_name no)
@@
 	(symbol
 		(lib_id "db:diode/05.035.0031.0002")
-		(at 199.39 72.39 270)
+		(at 209.55 72.39 270)
 		(unit 1)
 		(body_style 1)
@@
 		(fields_autoplaced yes)
 		(property "Reference" "D104"
-			(at 202.819 72.1303 90)
+			(at 212.979 72.1303 90)
 			(show_name no)
 			(do_not_autoplace no)
@@
 		)
 		(property "Value" "Green"
-			(at 202.819 74.5546 90)
+			(at 212.979 74.5546 90)
 			(show_name no)
 			(do_not_autoplace no)
@@
 		)
 		(property "Footprint" "diode:D_0603"
-			(at 199.39 72.39 90)
+			(at 209.55 72.39 90)
 			(hide yes)
 			(show_name no)
@@
 		)
 		(property "Datasheet" "${KICAD_USER_DATASHEET_DIR}diode/DS_LITEON_LTST-C190GKT.pdf"
-			(at 199.39 72.39 90)
+			(at 209.55 72.39 90)
 			(hide yes)
 			(show_name no)
@@
 		)
 		(property "Description" "Green LED"
-			(at 194.945 72.39 0)
+			(at 205.105 72.39 0)
 			(hide yes)
 			(show_name no)
@@
 		)
 		(property "Category" "diode"
-			(at 199.39 72.39 0)
+			(at 209.55 72.39 0)
 			(hide yes)
 			(show_name no)
@@
 		)
 		(property "MFR" "Lite-On"
-			(at 199.39 72.39 0)
+			(at 209.55 72.39 0)
 			(hide yes)
 			(show_name no)
@@
 		)
 		(property "Series" "LTST"
-			(at 199.39 72.39 0)
+			(at 209.55 72.39 0)
 			(hide yes)
 			(show_name no)
@@
 		)
 		(property "MFR#" "LTST-C190GKT"
-			(at 199.39 72.39 0)
+			(at 209.55 72.39 0)
 			(hide yes)
 			(show_name no)
@@
 		)
 		(property "Rating" "2v1 20mA 569nm"
-			(at 199.39 72.39 0)
+			(at 209.55 72.39 0)
 			(hide yes)
 			(show_name no)
@@
 		)
 		(property "Remarks" ""
-			(at 199.39 72.39 0)
+			(at 209.55 72.39 0)
 			(hide yes)
 			(show_name no)
@@
 		)
 		(property "Dist1" "digikey"
-			(at 199.39 72.39 0)
+			(at 209.55 72.39 0)
 			(hide yes)
 			(show_name no)
@@
 		)
 		(property "Dist1#" "160-LTST-C190GKTCT-ND"
-			(at 199.39 72.39 0)
+			(at 209.55 72.39 0)
 			(hide yes)
 			(show_name no)
@@
 		)
 		(property "Dist2" "mouser"
-			(at 199.39 72.39 0)
+			(at 209.55 72.39 0)
 			(hide yes)
 			(show_name no)
@@
 		)
 		(property "Dist2#" "859-LTST-C190GKT"
-			(at 199.39 72.39 0)
+			(at 209.55 72.39 0)
 			(hide yes)
 			(show_name no)
@@
 		)
 		(property "Dist3" "none"
-			(at 199.39 72.39 0)
+			(at 209.55 72.39 0)
 			(hide yes)
 			(show_name no)
@@
 		)
 		(property "Dist3#" ""
-			(at 199.39 72.39 0)
+			(at 209.55 72.39 0)
 			(hide yes)
 			(show_name no)
@@
 		)
 		(property "Active" "1"
-			(at 199.39 72.39 0)
+			(at 209.55 72.39 0)
 			(hide yes)
 			(show_name no)
@@
 		)
 		(property "Version" "2"
-			(at 199.39 72.39 0)
+			(at 209.55 72.39 0)
 			(hide yes)
 			(show_name no)
@@
 		)
 		(property "Modified" "2026-03-31 22:36:44"
-			(at 199.39 72.39 0)
+			(at 209.55 72.39 0)
 			(hide yes)
 			(show_name no)
@@
 		)
 		(property "FP" "D_0603"
-			(at 199.39 72.39 0)
+			(at 209.55 72.39 0)
 			(hide yes)
 			(show_name no)
@@
 	(symbol
 		(lib_id "db:resistor/00.018.0009.0005")
-		(at 199.39 66.04 0)
+		(at 209.55 66.04 0)
 		(unit 1)
 		(body_style 1)
@@
 		(fields_autoplaced yes)
 		(property "Reference" "R115"
-			(at 200.914 64.8278 0)
+			(at 211.074 64.8278 0)
 			(show_name no)
 			(do_not_autoplace no)
@@
 		)
 		(property "Value" "1k"
-			(at 200.914 67.2521 0)
+			(at 211.074 67.2521 0)
 			(show_name no)
 			(do_not_autoplace no)
@@
 		)
 		(property "Footprint" "passive:R_0603"
-			(at 199.39 66.04 0)
+			(at 209.55 66.04 0)
 			(hide yes)
 			(show_name no)
@@
 		)
 		(property "Datasheet" "${KICAD_USER_DATASHEET_DIR}passive/DS_Resistors_Yageo.pdf"
-			(at 199.39 66.04 0)
+			(at 209.55 66.04 0)
 			(hide yes)
 			(show_name no)
@@
 		)
 		(property "Description" ""
-			(at 199.39 66.04 0)
+			(at 209.55 66.04 0)
 			(hide yes)
 			(show_name no)
@@
 		)
 		(property "Category" "resistor"
-			(at 199.39 66.04 0)
+			(at 209.55 66.04 0)
 			(hide yes)
 			(show_name no)
@@
 		)
 		(property "MFR" "Yageo"
-			(at 199.39 66.04 0)
+			(at 209.55 66.04 0)
 			(hide yes)
 			(show_name no)
@@
 		)
 		(property "Series" "RC_L "
-			(at 199.39 66.04 0)
+			(at 209.55 66.04 0)
 			(hide yes)
 			(show_name no)
@@
 		)
 		(property "MFR#" "RC0603FR-071KL"
-			(at 199.39 66.04 0)
+			(at 209.55 66.04 0)
 			(hide yes)
 			(show_name no)
@@
 		)
 		(property "Rating" "100mW, 1%"
-			(at 199.39 66.04 0)
+			(at 209.55 66.04 0)
 			(hide yes)
 			(show_name no)
@@
 		)
 		(property "Remarks" ""
-			(at 199.39 66.04 0)
+			(at 209.55 66.04 0)
 			(hide yes)
 			(show_name no)
@@
 		)
 		(property "Dist1" "digikey"
-			(at 199.39 66.04 0)
+			(at 209.55 66.04 0)
 			(hide yes)
 			(show_name no)
@@
 		)
 		(property "Dist1#" "311-1.00KHRCT-ND"
-			(at 199.39 66.04 0)
+			(at 209.55 66.04 0)
 			(hide yes)
 			(show_name no)
@@
 		)
 		(property "Dist2" "none"
-			(at 199.39 66.04 0)
+			(at 209.55 66.04 0)
 			(hide yes)
 			(show_name no)
@@
 		)
 		(property "Dist2#" ""
-			(at 199.39 66.04 0)
+			(at 209.55 66.04 0)
 			(hide yes)
 			(show_name no)
@@
 		)
 		(property "Dist3" "none"
-			(at 199.39 66.04 0)
+			(at 209.55 66.04 0)
 			(hide yes)
 			(show_name no)
@@
 		)
 		(property "Dist3#" ""
-			(at 199.39 66.04 0)
+			(at 209.55 66.04 0)
 			(hide yes)
 			(show_name no)
@@
 		)
 		(property "Active" "1"
-			(at 199.39 66.04 0)
+			(at 209.55 66.04 0)
 			(hide yes)
 			(show_name no)
@@
 		)
 		(property "Version" "1"
-			(at 199.39 66.04 0)
+			(at 209.55 66.04 0)
 			(hide yes)
 			(show_name no)
@@
 		)
 		(property "Modified" "2026-02-11 09:17:49"
-			(at 199.39 66.04 0)
+			(at 209.55 66.04 0)
 			(hide yes)
 			(show_name no)
@@
 		)
 		(property "FP" "R_0603"
-			(at 199.39 66.04 0)
+			(at 209.55 66.04 0)
 			(hide yes)
 			(show_name no)
