File: mpht_usb.kicad_sch (KiCad schematic)
At the start: 8 parts, among them J101 USB4105GFA120, U101 RCLAMP0854P.TCT

Commit message: Added On/Off Switch Mode Selection Added a List of ToDos
Other:
- note removed: "USB-C Receptecal"
- moved on the sheet: J101, L102, L103, R101, R102, R103, R104, U101
