File: MPHT.kicad_pcb (KiCad board)
At the start: 2 copper layers, 0 parts

Commit message: Created hierarchical sheets for MCU, BMS and USB Organized components roughly on PCB
Parts:
- added BT3: AAA-Battery Holder (Left Version), misc:battery_holder_aaa_right_angle_left, F.Cu at (123.3, 107.5)
- added BT4: AAA-Battery Holder (Right Version), misc:battery_holder_aaa_right_angle_right, F.Cu at (179.9, 107.5)
- added C1: 1u, passive:C_0603, F.Cu at (137.7, 91.7)
- added C109: 4u7, passive:C_0603, F.Cu at (180.9, 92.3)
- added C2: 1u, passive:C_0603, F.Cu at (172.0, 108.7)
- added C3: 1u, passive:C_0603, F.Cu at (176.5, 96.1)
- added C4: 10u, passive:C_0603, F.Cu at (180.9, 95.2)
- added C5: 10u, passive:C_0603, F.Cu at (179.2, 99.3)
- added C6: 22p, passive:C_0603, F.Cu at (186.0, 102.9)
- added C7: 10u, passive:C_0603, F.Cu at (182.9, 102.9)
- added C8: 470n, passive:C_0603, F.Cu at (174.4, 96.1)
- added C9: 10u, passive:C_0603, F.Cu at (182.5, 97.4)
- added D1: Orange, diode:D_0603, F.Cu at (169.0, 130.9)
- added D104: Green, diode:D_0603, F.Cu at (161.7, 110.4)
- added J101: USB4105GFA120, connector:GCT_USB4105GFA120, F.Cu at (157.7, 130.8)
- added L102: 330, passive:L_0603, F.Cu at (164.8, 130.7)
- added L103: 330, passive:L_0603, F.Cu at (162.9, 124.0)
- added L2: 2u2, passive:L_3.2mmx2.5mm, F.Cu at (180.1, 105.3)
- added R1: 10k, passive:R_0603, F.Cu at (140.5, 94.2)
- added R101: 5k1, passive:R_0603, F.Cu at (165.7, 127.6)
- added R102: 5k1, passive:R_0603, F.Cu at (164.1, 127.5)
- added R103: 33, passive:R_0603, F.Cu at (145.5, 105.4)
- added R104: 33, passive:R_0603, F.Cu at (145.5, 106.8)
- added R107: 10k, passive:R_0603, F.Cu at (169.0, 108.7)
- added R11: 10k, passive:R_0603, F.Cu at (184.2, 97.4)
- added R115: 1k, passive:R_0603, F.Cu at (164.9, 110.5)
- added R12: 13k, passive:R_0603, F.Cu at (183.4, 88.4)
- added R13: 10k, passive:R_0603, F.Cu at (185.2, 92.0)
- added R14: 604R, passive:R_0603, F.Cu at (182.0, 88.4)
- added R15: 619k, passive:R_0603, F.Cu at (184.6, 102.9)
- added R16: 137k, passive:R_0603, F.Cu at (183.7, 100.2)
- added R17: 10k, passive:R_0603, F.Cu at (184.8, 88.4)
- added R18: 10k, passive:R_0603, F.Cu at (169.0, 129.4)
- added R19: 10k, passive:R_0603, F.Cu at (173.1, 89.0)
- added R2: 4k7, passive:R_0603, F.Cu at (145.5, 95.9)
- added R20: 10m, passive:R_0603, F.Cu at (176.3, 88.5)
- added R3: 4k7, passive:R_0603, F.Cu at (142.8, 97.1)
- added SW101: KMR421GULCLFS, switch:KMR421GULCLFS, F.Cu at (171.9, 106.0)
- added SW102: KMR421GULCLFS, switch:KMR421GULCLFS, F.Cu at (141.7, 91.7)
- added U1: ESP32-S3-WROOM-1-N4R2, mcu:ESP32_S3_WROOM_1, F.Cu at (157.6, 95.6)
- added U101: RCLAMP0854P.TCT, package:UFDFN06_1P6X1P6, F.Cu at (159.4, 123.0)
- added U4: TPS62590, package:WSON-6-1EP_2x2mm_P0.65mm, F.Cu at (180.0, 101.7)
- added U5: BQ25185, package:WSON-10-1EP_2.2x2mm_P0.4mm, F.Cu at (182.9, 93.8)
- added U6: BQ27441-G1, package:VSON-12-1EP_2.5_4mm_P0.4mm, F.Cu at (174.8, 92.4)
Other:
- board outline added: 60 x 50 mm

Commit message: Added On/Off Switch Mode Selection Added a List of ToDos
Parts:
- added R4: 0, passive:R_0603_DNP, F.Cu at (145.8, 126.6)
- added R5: 0, passive:R_0603, F.Cu at (149.3, 128.4)
- added R6: 10k, passive:R_0603, F.Cu at (149.3, 130.2)
- added R8: 0, passive:R_0603_DNP, F.Cu at (145.8, 130.2)
- added R9: 0, passive:R_0603_DNP, F.Cu at (145.8, 128.4)
Connections:
- U1 pad 10: unconnected-(U1-IO17-Pad10) -> /MCU/SLEEP_CTRL_PIN
- U4 pad 4: VSYS -> /Buck_En

Commit message: Replace placeholder switch symbol with actual symbol Adjusted max charge current to match new batteries
Parts:
- added SW1: OS102011MA1QN1, switch:OS102011MA1QN1_CNK, F.Cu at (147.1, 129.7)
- R14: value 604R -> 768R
- moved R8 8.43 mm to (152.6, 125.1), turned to -90 degrees
- moved R102 6.83 mm to (169.4, 123.3)
- moved L102 6.83 mm to (170.2, 126.5)
- moved R101 6.83 mm to (171.1, 123.3)
- moved R6 6.41 mm to (145.4, 125.1), turned to -90 degrees
- moved R9 6.10 mm to (150.9, 125.1), turned to -90 degrees
- moved J101 4.24 mm to (161.9, 130.8)
- moved R5 3.92 mm to (147.2, 125.1), turned to -90 degrees
- moved R4 3.57 mm to (149.0, 125.1), turned to 90 degrees
- moved R18 0.99 mm to (170.0, 129.4)
- moved D1 0.88 mm to (169.9, 131.0)
Other:
- board text added: "Buck:10k|0|-|-|- MCU: -|-|0|0|10k"
