File: MPHT.kicad_sch (KiCad schematic)
At the start: 0 parts

Commit message: Created hierarchical sheets for MCU, BMS and USB Organized components roughly on PCB
Other:
- added sheet BMS (mpht_bms.kicad_sch)
- added sheet MCU (mpht_mcu.kicad_sch)
- added sheet USB (mpht_usb.kicad_sch)

Commit message: Added On/Off Switch Mode Selection Added a List of ToDos
Parts:
- added R4, R8, R9: 0, passive:R_0603_DNP, symbol db:resistor/00.000.0000.0002
- added R5: 0, passive:R_0603, symbol db:resistor/00.000.0000.0001
- added R6: 10k, passive:R_0603, symbol db:resistor/00.018.0009.0006
- added SW2: SW_SPDT, symbol Switch:SW_SPDT
Connections:
- new net: R6.2, R8.2, SW2.1 (A)
- new net: R4.2, R5.2, SW2.2 (B)
- new net +3V3: R8.1
- new net Buck_En: R5.1, R9.2
- new net GND: SW2.3 (C)
- new net MCU/SLEEP_CTRL_PIN: R4.1
- new net VSYS: R6.1, R9.1
Other:
- sheet BMS ports: added BUCK_EN; removed none
- sheet MCU ports: added SLEEP_CTRL_PIN; removed none
- note added: "Select On/Off Type: - Buck Shutdown: R6 10k, R5 0 - MCU Shutdown: R8 10k, R4 0, R9 0"
- note added: "ToDos: - Mounting Holes - Real Time Clock Module - Control Switch - Replace On/Off Switch with correct symbol - Display - Replace Power LED with right angle variant - Check Current limits for Charger for the new batteries - Maybe a Buzzer"

Commit message: Replace placeholder switch symbol with actual symbol Adjusted max charge current to match new batteries
Parts:
- removed SW2: SW_SPDT, symbol Switch:SW_SPDT
- added SW1: OS102011MA1QN1, switch:OS102011MA1QN1_CNK, symbol db:switch/06.004.0051.0001
Connections:
- net GND: now also SW1.3 (C)
- net at R6.2, R8.2: now also SW1.1 (A)
- net at R4.2, R5.2: now also SW1.2 (B)
Other:
- note added: "ToDos: - Mounting Holes - Real Time Clock Module - Control Switch - Display - Replace Power LED with right angle variant - Maybe a Buzzer"
- note removed: "ToDos: - Mounting Holes - Real Time Clock Module - Control Switch - Replace On/Off Switch with correct symbol - Display - Replace Power LED with right angle variant - Check Current limits for Charger for the new batteries - Maybe a Buzzer"
Changed lines of the file:
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@@
 		)
 	)
-	(text "ToDos:\n- Mounting Holes\n- Real Time Clock Module\n- Control Switch\n- Replace On/Off Switch with correct symbol\n- Display\n- Replace Power LED with right angle variant\n- Check Current limits for Charger for the new batteries\n- Maybe a Buzzer"
+	(text "ToDos:\n- Mounting Holes\n- Real Time Clock Module\n- Control Switch\n- Display\n- Replace Power LED with right angle variant\n- Maybe a Buzzer"
 		(exclude_from_sim no)
 		(at 48.006 133.604 0)
@@
 	)
 	(symbol
+		(lib_id "db:switch/06.004.0051.0001")
+		(at 209.55 90.17 0)
+		(unit 1)
+		(body_style 1)
+		(exclude_from_sim no)
+		(in_bom yes)
+		(on_board yes)
+		(in_pos_files yes)
+		(dnp no)
+		(fields_autoplaced yes)
+		(property "Reference" "SW1"
+			(at 209.55 82.3425 0)
+			(show_name no)
+			(do_not_autoplace no)
+			(effects
+				(font
+					(size 1.27 1.27)
+				)
+			)
+		)
+		(property "Value" "OS102011MA1QN1"
+			(at 209.55 84.7668 0)
+			(show_name no)
+			(do_not_autoplace no)
+			(effects
+				(font
+					(size 1.27 1.27)
+				)
+			)
+		)
+		(property "Footprint" "switch:OS102011MA1QN1_CNK"
+			(at 209.55 90.17 0)
+			(hide yes)
+			(show_name no)
+			(do_not_autoplace no)
+			(effects
+				(font
+					(size 1.27 1.27)
+				)
+			)
+		)
+		(property "Datasheet" "${KICAD_USER_DATASHEET_DIR}switch/DS_CK_OS_Series.pdf"
+			(at 209.55 97.79 0)
+			(hide yes)
+			(show_name no)
+			(do_not_autoplace no)
+			(effects
+				(font
+					(size 1.27 1.27)
+				)
+			)
+		)
+		(property "Description" ""
+			(at 209.55 90.17 0)
+			(hide yes)
+			(show_name no)
+			(do_not_autoplace no)
+			(effects
+				(font
+					(size 1.27 1.27)
+				)
+			)
+		)
+		(property "Category" "switch"
+			(at 209.55 90.17 0)
+			(hide yes)
+			(show_name no)
+			(do_not_autoplace no)
+			(effects
+				(font
+					(size 1.27 1.27)
+				)
+			)
+		)
+		(property "MFR" "C&K"
+			(at 209.55 90.17 0)
+			(hide yes)
+			(show_name no)
+			(do_not_autoplace no)
+			(effects
+				(font
+					(size 1.27 1.27)
+				)
+			)
+		)
+		(property "Series" "OS"
+			(at 209.55 90.17 0)
+			(hide yes)
+			(show_name no)
+			(do_not_autoplace no)
+			(effects
+				(font
+					(size 1.27 1.27)
+				)
+			)
+		)
+		(property "MFR#" "OS102011MA1QN1"
+			(at 209.55 90.17 0)
+			(hide yes)
+			(show_name no)
+			(do_not_autoplace no)
+			(effects
+				(font
+					(size 1.27 1.27)
+				)
+			)
+		)
+		(property "Rating" "100MA 12V Non-shorting"
+			(at 209.55 90.17 0)
+			(hide yes)
+			(show_name no)
+			(do_not_autoplace no)
+			(effects
+				(font
+					(size 1.27 1.27)
+				)
+			)
+		)
+		(property "Remarks" ""
+			(at 209.55 90.17 0)
+			(hide yes)
+			(show_name no)
+			(do_not_autoplace no)
+			(effects
+				(font
+					(size 1.27 1.27)
+				)
+			)
+		)
+		(property "Dist1" "digikey"
+			(at 209.55 90.17 0)
+			(hide yes)
+			(show_name no)
+			(do_not_autoplace no)
+			(effects
+				(font
+					(size 1.27 1.27)
+				)
+			)
+		)
+		(property "Dist1#" "CKN9559-ND"
+			(at 209.55 90.17 0)
+			(hide yes)
+			(show_name no)
+			(do_not_autoplace no)
+			(effects
+				(font
+					(size 1.27 1.27)
+				)
+			)
+		)
+		(property "Dist2" "none"
+			(at 209.55 90.17 0)
+			(hide yes)
+			(show_name no)
+			(do_not_autoplace no)
+			(effects
+				(font
+					(size 1.27 1.27)
+				)
+			)
+		)
+		(property "Dist2#" ""
+			(at 209.55 90.17 0)
+			(hide yes)
+			(show_name no)
+			(do_not_autoplace no)
+			(effects
+				(font
+					(size 1.27 1.27)
+				)
+			)
+		)
+		(property "Dist3" "none"
+			(at 209.55 90.17 0)
+			(hide yes)
+			(show_name no)
+			(do_not_autoplace no)
+			(effects
+				(font
+					(size 1.27 1.27)
+				)
+			)
+		)
+		(property "Dist3#" ""
+			(at 209.55 90.17 0)
+			(hide yes)
+			(show_name no)
+			(do_not_autoplace no)
+			(effects
+				(font
+					(size 1.27 1.27)
+				)
+			)
+		)
+		(property "Active" "1"
+			(at 209.55 90.17 0)
+			(hide yes)
+			(show_name no)
+			(do_not_autoplace no)
+			(effects
+				(font
+					(size 1.27 1.27)
+				)
+			)
+		)
+		(property "Version" "2"
+			(at 209.55 90.17 0)
+			(hide yes)
+			(show_name no)
+			(do_not_autoplace no)
+			(effects
+				(font
+					(size 1.27 1.27)
+				)
+			)
+		)
+		(property "Modified" "2026-10-05 20:13:12"
+			(at 209.55 90.17 0)
+			(hide yes)
+			(show_name no)
+			(do_not_autoplace no)
+			(effects
+				(font
+					(size 1.27 1.27)
+				)
+			)
+		)
+		(property "FP" "OS102011MA1QN1_CNK"
+			(at 209.55 90.17 0)
+			(hide yes)
+			(show_name no)
+			(do_not_autoplace no)
+			(effects
+				(font
+					(size 1.27 1.27)
+				)
+			)
+		)
+		(pin "3"
+		)
+		(pin "1"
+		)
+		(pin "2"
+		)
+		(instances
+			(project "MPHT"
+				(path "/328ebaa0-d01b-4b80-b614-bb0154e8d306"
+					(reference "SW1")
+					(unit 1)
+				)
+			)
+		)
+	)
+	(symbol
 		(lib_name "resistor/00.000.0000.0002_1")
 		(lib_id "db:resistor/00.000.0000.0002")
@@
 					(unit 1)
 				)
-			)
-		)
-	)
-	(symbol
-		(lib_id "Switch:SW_SPDT")
-		(at 209.55 90.17 0)
-		(unit 1)
-		(body_style 1)
-		(exclude_from_sim no)
-		(in_bom yes)
-		(on_board yes)
-		(in_pos_files yes)
-		(dnp no)
-		(fields_autoplaced yes)
-		(property "Reference" "SW2"
-			(at 209.55 82.3425 0)
-			(show_name no)
-			(do_not_autoplace no)
-			(effects
-				(font
-					(size 1.27 1.27)
-				)
-			)
-		)
-		(property "Value" "SW_SPDT"
-			(at 209.55 84.7668 0)
-			(show_name no)
-			(do_not_autoplace no)
-			(effects
-				(font
-					(size 1.27 1.27)
-				)
-			)
-		)
-		(property "Footprint" ""
-			(at 209.55 90.17 0)
-			(hide yes)
-			(show_name no)
-			(do_not_autoplace no)
-			(effects
-				(font
-					(size 1.27 1.27)
-				)
-			)
-		)
-		(property "Datasheet" ""
-			(at 209.55 97.79 0)
-			(hide yes)
-			(show_name no)
-			(do_not_autoplace no)
-			(effects
-				(font
-					(size 1.27 1.27)
-				)
-			)
-		)
-		(property "Description" "Switch, single pole double throw"
-			(at 209.55 90.17 0)
-			(hide yes)
-			(show_name no)
-			(do_not_autoplace no)
-			(effects
-				(font
-					(size 1.27 1.27)
-				)
-			)
-		)
-		(pin "2"
-		)
-		(pin "3"
-		)
-		(pin "1"
-		)
-		(instances
-			(project "MPHT"
-				(path "/328ebaa0-d01b-4b80-b614-bb0154e8d306"
-					(reference "SW2")
-					(unit 1)
-				)
