File: mpht_bms.kicad_sch (KiCad schematic)
At the start: 25 parts, among them U4 TPS62590, U5 BQ25185, U6 BQ27441-G1

Commit message: Added On/Off Switch Mode Selection Added a List of ToDos
Connections:
- net VSYS: no longer U4.4 (EN)
- new net BUCK_EN: U4.4 (EN)
Other:
- note added: "1100mA in current limit +4V2 Battery Voltage"
- note removed: "1100mA in current limit 4V2 Battery Voltage"
- note removed: "Check limits again"
- moved on the sheet: C5
Changed lines of the file:
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@@
 		)
 	)
-	(text "Check limits again\n"
-		(exclude_from_sim no)
-		(at 31.75 66.548 0)
-		(effects
-			(font
-				(size 1.27 1.27)
-			)
-		)
-	)
 	(text "Fuel Gauge\n"
 		(exclude_from_sim no)
@@
 		)
 	)
-	(text "1100mA in current limit\n4V2 Battery Voltage"
+	(text "1100mA in current limit\n+4V2 Battery Voltage"
 		(exclude_from_sim no)
 		(at 64.516 68.834 0)
@@
 	)
 	(junction
-		(at 60.96 105.41)
-		(diameter 0)
-		(color 0 0 0 0)
-	)
-	(junction
-		(at 72.39 105.41)
+		(at 55.88 105.41)
 		(diameter 0)
 		(color 0 0 0 0)
@@
 	)
 	(junction
-		(at 60.96 113.03)
+		(at 55.88 113.03)
 		(diameter 0)
 		(color 0 0 0 0)
@@
 	(wire
 		(pts
-			(xy 60.96 113.03) (xy 60.96 124.46)
+			(xy 55.88 113.03) (xy 55.88 124.46)
 		)
 		(stroke
@@
 	(wire
 		(pts
-			(xy 72.39 105.41) (xy 72.39 109.22)
-		)
-		(stroke
-			(width 0)
-			(type default)
-		)
-	)
-	(wire
-		(pts
 			(xy 116.84 111.76) (xy 116.84 113.03)
 		)
@@
 	(wire
 		(pts
-			(xy 55.88 105.41) (xy 60.96 105.41)
+			(xy 55.88 105.41) (xy 77.47 105.41)
 		)
 		(stroke
@@
 	(wire
 		(pts
-			(xy 60.96 113.03) (xy 77.47 113.03)
+			(xy 55.88 113.03) (xy 77.47 113.03)
 		)
 		(stroke
@@
 	(wire
 		(pts
-			(xy 60.96 105.41) (xy 60.96 106.68)
+			(xy 55.88 105.41) (xy 55.88 106.68)
 		)
 		(stroke
@@
 	(wire
 		(pts
-			(xy 72.39 105.41) (xy 77.47 105.41)
-		)
-		(stroke
-			(width 0)
-			(type default)
-		)
-	)
-	(wire
-		(pts
 			(xy 134.62 49.53) (xy 132.08 49.53)
 		)
@@
 	(wire
 		(pts
-			(xy 60.96 105.41) (xy 72.39 105.41)
-		)
-		(stroke
-			(width 0)
-			(type default)
-		)
-	)
-	(wire
-		(pts
 			(xy 105.41 109.22) (xy 105.41 113.03)
 		)
@@
 	(wire
 		(pts
-			(xy 60.96 111.76) (xy 60.96 113.03)
+			(xy 55.88 111.76) (xy 55.88 113.03)
 		)
 		(stroke
@@
 		)
 	)
+	(hierarchical_label "BUCK_EN"
+		(shape input)
+		(at 72.39 109.22 180)
+		(effects
+			(font
+				(size 1.27 1.27)
+			)
+			(justify right)
+		)
+	)
 	(hierarchical_label "CHRG_STAT1"
 		(shape output)
@@
 	(symbol
 		(lib_id "power:GND")
-		(at 60.96 124.46 0)
+		(at 55.88 124.46 0)
 		(unit 1)
 		(body_style 1)
@@
 		(fields_autoplaced yes)
 		(property "Reference" "#PWR023"
-			(at 60.96 130.81 0)
+			(at 55.88 130.81 0)
 			(hide yes)
 			(show_name no)
@@
 		)
 		(property "Value" "GND"
-			(at 60.96 128.5931 0)
+			(at 55.88 128.5931 0)
 			(hide yes)
 			(show_name no)
@@
 		)
 		(property "Footprint" ""
-			(at 60.96 124.46 0)
+			(at 55.88 124.46 0)
 			(hide yes)
 			(show_name no)
@@
 		)
 		(property "Datasheet" ""
-			(at 60.96 124.46 0)
+			(at 55.88 124.46 0)
 			(hide yes)
 			(show_name no)
@@
 		)
 		(property "Description" "Power symbol creates a global label with name \"GND\" , ground"
-			(at 60.96 124.46 0)
+			(at 55.88 124.46 0)
 			(hide yes)
 			(show_name no)
@@
 	(symbol
 		(lib_id "db:capacitor/01.018.0008.0001")
-		(at 60.96 109.22 0)
+		(at 55.88 109.22 0)
 		(unit 1)
 		(body_style 1)
@@
 		(fields_autoplaced yes)
 		(property "Reference" "C5"
-			(at 62.9285 108.0078 0)
+			(at 57.8485 108.0078 0)
 			(show_name no)
 			(do_not_autoplace no)
@@
 		)
 		(property "Value" "10u"
-			(at 62.9285 110.4321 0)
+			(at 57.8485 110.4321 0)
 			(show_name no)
 			(do_not_autoplace no)
@@
 		)
 		(property "Footprint" "passive:C_0603"
-			(at 60.96 109.22 0)
+			(at 55.88 109.22 0)
 			(hide yes)
 			(show_name no)
@@
 		)
 		(property "Datasheet" "${KICAD_USER_DATASHEET_DIR}passive/DS_CC0603MRX5R6BB106.pdf"
-			(at 60.96 109.22 0)
+			(at 55.88 109.22 0)
 			(hide yes)
 			(show_name no)
@@
 		)
 		(property "Description" "MLCC"
-			(at 60.96 109.22 0)
+			(at 55.88 109.22 0)
 			(hide yes)
 			(show_name no)
@@
 		)
 		(property "Category" "capacitor"
-			(at 60.96 109.22 0)
+			(at 55.88 109.22 0)
 			(hide yes)
 			(show_name no)
@@
 		)
 		(property "MFR" "Yageo"
-			(at 60.96 109.22 0)
+			(at 55.88 109.22 0)
 			(hide yes)
 			(show_name no)
@@
 		)
 		(property "Series" "CC-X5R"
-			(at 60.96 109.22 0)
+			(at 55.88 109.22 0)
 			(hide yes)
 			(show_name no)
@@
 		)
 		(property "MFR#" "CC0603MRX5R6BB106"
-			(at 60.96 109.22 0)
+			(at 55.88 109.22 0)
 			(hide yes)
 			(show_name no)
@@
 		)
 		(property "Rating" "10V 20%"
-			(at 60.96 109.22 0)
+			(at 55.88 109.22 0)
 			(hide yes)
 			(show_name no)
@@
 		)
 		(property "Remarks" ""
-			(at 60.96 109.22 0)
+			(at 55.88 109.22 0)
 			(hide yes)
 			(show_name no)
@@
 		)
 		(property "Dist1" "digikey"
-			(at 60.96 109.22 0)
+			(at 55.88 109.22 0)
 			(hide yes)
 			(show_name no)
@@
 		)
 		(property "Dist1#" "311-1817-1-ND"
-			(at 60.96 109.22 0)
+			(at 55.88 109.22 0)
 			(hide yes)
 			(show_name no)
@@
 		)
 		(property "Dist2" "none"
-			(at 60.96 109.22 0)
+			(at 55.88 109.22 0)
 			(hide yes)
 			(show_name no)
@@
 		)
 		(property "Dist2#" ""
-			(at 60.96 109.22 0)
+			(at 55.88 109.22 0)
 			(hide yes)
 			(show_name no)
@@
 		)
 		(property "Dist3" "none"
-			(at 60.96 109.22 0)
+			(at 55.88 109.22 0)
 			(hide yes)
 			(show_name no)
@@
 		)
 		(property "Dist3#" ""
-			(at 60.96 109.22 0)
+			(at 55.88 109.22 0)
 			(hide yes)
 			(show_name no)
@@
 		)
 		(property "Active" "1"
-			(at 60.96 109.22 0)
+			(at 55.88 109.22 0)
 			(hide yes)
 			(show_name no)
@@
 		)
 		(property "Version" "1"
-			(at 60.96 109.22 0)
+			(at 55.88 109.22 0)
 			(hide yes)
 			(show_name no)
@@
 		)
 		(property "Modified" "2026-03-22 17:13:24"
-			(at 60.96 109.22 0)
+			(at 55.88 109.22 0)
 			(hide yes)
 			(show_name no)
@@
 		)
 		(property "FP" "C_0603"
-			(at 60.96 109.22 0)
+			(at 55.88 109.22 0)
 			(hide yes)
 			(show_name no)

Commit message: Replace placeholder switch symbol with actual symbol Adjusted max charge current to match new batteries
Parts:
- R14: value 604R -> 768R; symbol db:resistor/00.018.0009.0027 -> db:resistor/00.018.0009.0036; Dist1# 311-604HRCT-ND -> 311-768HRCT-ND; MFR# RC0603FR-07604RL -> RC0603FR-07768RL; Modified 2026-07-28 21:04:21 -> 2026-10-05 20:40:11; Version 3 -> 2
Other:
- note added: "390mA charge current limit"
- note removed: "500mA charge current limit"
Changed lines of the file:
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@@
 		)
 	)
-	(text "500mA charge current limit"
+	(text "390mA charge current limit"
 		(exclude_from_sim no)
 		(at 102.108 77.216 0)
@@
 	)
 	(symbol
-		(lib_id "db:resistor/00.018.0009.0027")
+		(lib_id "db:resistor/00.018.0009.0036")
 		(at 88.9 68.58 0)
 		(unit 1)
@@
 			)
 		)
-		(property "Value" "604R"
+		(property "Value" "768R"
 			(at 90.424 69.7921 0)
 			(show_name no)
@@
 			)
 		)
-		(property "MFR#" "RC0603FR-07604RL"
+		(property "MFR#" "RC0603FR-07768RL"
 			(at 88.9 68.58 0)
 			(hide yes)
@@
 			)
 		)
-		(property "Dist1#" "311-604HRCT-ND"
+		(property "Dist1#" "311-768HRCT-ND"
 			(at 88.9 68.58 0)
 			(hide yes)
@@
 			)
 		)
-		(property "Version" "3"
+		(property "Version" "2"
 			(at 88.9 68.58 0)
 			(hide yes)
@@
 			)
 		)
-		(property "Modified" "2026-07-28 21:04:21"
+		(property "Modified" "2026-10-05 20:40:11"
 			(at 88.9 68.58 0)
 			(hide yes)
