File: MPT.kicad_pcb (KiCad board)
At the start: 2 copper layers, 60 x 50 mm, 50 parts, among them J101 USB4105GFA120, SW1 OS102011MA1QN1, SW101 KMR421GULCLFS, SW102 KMR421GULCLFS, U1 ESP32-S3-WROOM-1-N4R2, U101 RCLAMP0854P.TCT, U4 TPS62590, U5 BQ25185, U6 BQ27441-G1

Commit message: Add Text on PCB for reset and boot button
Other:
- board text added: "BOOT"
- board text added: "RST"
Changed lines of the file:
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@@
 			(unlocked yes)
 			(layer "F.SilkS")
+			(hide yes)
 			(effects
 				(font
@@
 		(layer "Edge.Cuts")
 	)
+	(gr_text "RST"
+		(at 139.7 89.4842 0)
+		(layer "F.SilkS")
+		(effects
+			(font
+				(size 1.5 1.5)
+				(thickness 0.3)
+				(bold yes)
+			)
+			(justify left bottom)
+		)
+	)
+	(gr_text "BOOT"
+		(at 168.8338 103.759 0)
+		(layer "F.SilkS")
+		(effects
+			(font
+				(size 1.5 1.5)
+				(thickness 0.3)
+				(bold yes)
+			)
+			(justify left bottom)
+		)
+	)
 	(gr_text "Buck:10k|0|-|-|-\nMCU:   -|-|0|0|10k"

Commit message: Added Display
Parts:
- added J2: ER-TFT2.79-1, misc:ER-TFT2.79-1, F.Cu at (138.5, 100.8)
- added Q1: BSS138, package:SOT-23, F.Cu at (115.5, 113.4)
- added R26: 5R11, passive:R_0805, F.Cu at (111.2, 112.7)
- added R27: 100k, passive:R_0603, F.Cu at (107.0, 112.5)
- added R28: 100R, passive:R_0603, F.Cu at (107.0, 114.9)
- C2: renamed from C109; footprint passive:C_0603 -> passive:C_0805
- D1: value Orange -> Red; footprint diode:D_0603 -> diode:LED_0805_Right_Angle
- R21: renamed from R101; value 5k1 -> 5k11
- R22: renamed from R102; value 5k1 -> 5k11
- R23: renamed from R103; value 33 -> 33R2
- R24: renamed from R104; value 33 -> 33R2
- moved SW1 0.83 mm to (147.1, 128.9)
- moved C10 0.57 mm to (172.6, 108.7)
- moved R1 0.32 mm to (150.8, 124.8)
- moved R2 0.31 mm to (149.0, 124.8)
- moved R4 0.30 mm to (152.6, 124.8)
- moved R3 0.28 mm to (147.2, 124.8)
- moved D1 0.27 mm to (169.8, 131.3), turned to 0 degrees
- moved R5 0.27 mm to (145.4, 124.8)
- moved C8 0.13 mm to (176.6, 96.3)
- renumbered BT3 to BT1, BT4 to BT2, C5 to C1, C2 to C10, C6 to C3, C7 to C5, C9 to C6, C8 to C7, C3 to C8, C1 to C9, D104 to D2, J101 to J1, L2 to L1, L102 to L2, L103 to L3, R9 to R1, R15 to R10, R16 to R11, R17 to R12, R18 to R13, R19 to R14, R20 to R15, R1 to R16, R107 to R17, R2 to R18, R3 to R19, R4 to R2, R115 to R20, R5 to R3, R8 to R4, R6 to R5, R11 to R6, R12 to R7, R13 to R8, R14 to R9, SW102 to SW2, SW101 to SW3, U4 to U1, U5 to U2, U6 to U3, U1 to U4, U101 to U5
Connections:
- J1 pad A7: Net-(J101-DN1) -> Net-(J1-DN1)
- J1 pad B7: Net-(J101-DN1) -> Net-(J1-DN1)
- R16 pad 1: +3V3 -> /MCU/Chip Enable/Reset
- R16 pad 2: /MCU/Chip Enable/Reset -> +3V3
- R24 pad 1: Net-(J101-DN1) -> /MCU/USB_DP
- R24 pad 2: /MCU/USB_DP -> Net-(J1-DN1)
- SW1 pad 4: (no net) -> GND
- U1 pad 4: /Buck_En -> /BUCK_EN
- U1 pad 7: (no net) -> GND
- U4 pad 12: /MCU/DISP_BACKLIGHT -> /Display/DISP_BACKLIGHT
- U4 pad 17: /MCU/SPI2_SCL -> /Display/SPI2_SCL
- U4 pad 18: /MCU/SPI2_SDA0 -> /Display/SPI2_SDA
- U4 pad 19: /MCU/SPI2_SDA1 -> /Display/SPI2_CS0_DISP
- U4 pad 20: /MCU/SPI2_SDA2 -> /Display/DISP_RS
- U4 pad 21: /MCU/SPI2_SDA3 -> /Display/DISP_RESET
- U4 pad 22: /MCU/SPI2_CS0_DISP -> unconnected-(U4-IO14-Pad22)
- U5 pad 1: Net-(J101-DN1) -> Net-(J1-DN1)
Other:
- outline, holes or cut-outs redrawn
