File: mpt_display.kicad_sch (KiCad schematic)
At the start: 5 parts, among them J2 ER-TFT2.79-1, Q1 BSS138

Commit message: Work in Progress of RTC Added Sheet Titles
Other:
- company: (none) -> Hochschule Luzern, Technik & Architektur
- title: (none) -> M.P.T Display
Changed lines of the file:
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@@
 	(generator_version "10.0")
 	(paper "A4")
+	(title_block
+		(title "M.P.T Display")
+		(company "Hochschule Luzern, Technik & Architektur")
+	)
 	(junction
 		(at 191.77 116.84)
