File: mpt_mcu.kicad_sch (KiCad schematic)
At the start: 11 parts, among them SW101 KMR421GULCLFS, SW102 KMR421GULCLFS, U1 ESP32-S3-WROOM-1-N4R2

Commit message: Added Display
Parts:
- C10: renamed from C2; symbol db:capacitor/01.018.0025.0002 -> db:capacitor/01.018.0025.0013; Dist1# 311-1446-1-ND -> 311-2082-1-ND; MFR# CC0603KRX7R7BB105 -> CC0603KRX7R9BB105; Modified 2026-03-22 17:11:33 -> 2026-10-07 18:52:36; Rating 16V 10% -> 50V 10%
- C9: renamed from C1; symbol db:capacitor/01.018.0025.0002 -> db:capacitor/01.018.0025.0013; Dist1# 311-1446-1-ND -> 311-2082-1-ND; MFR# CC0603KRX7R7BB105 -> CC0603KRX7R9BB105; Modified 2026-03-22 17:11:33 -> 2026-10-07 18:52:36; Rating 16V 10% -> 50V 10%
- R16: renamed from R1; symbol db:resistor/00.018.0009.0006 -> db:resistor_0603/00.018.0009.0046; Modified 2026-02-11 09:36:06 -> 2026-10-07 14:47:41; Rating 100mW, 1% -> 125mW, 1%; Remarks (none) -> Autogenerated
- R17: renamed from R107; symbol db:resistor/00.018.0009.0006 -> db:resistor_0603/00.018.0009.0046; Modified 2026-02-11 09:36:06 -> 2026-10-07 14:47:41; Rating 100mW, 1% -> 125mW, 1%; Remarks (none) -> Autogenerated
- R18: renamed from R2; symbol db:resistor/00.018.0009.0035 -> db:resistor_0603/00.018.0009.0035
- R19: renamed from R3; symbol db:resistor/00.018.0009.0035 -> db:resistor_0603/00.018.0009.0035
- R20: renamed from R115; symbol db:resistor/00.018.0009.0005 -> db:resistor_0603/00.018.0009.0045; Modified 2026-02-11 09:17:49 -> 2026-10-07 14:47:41; Rating 100mW, 1% -> 125mW, 1%; Remarks (none) -> Autogenerated; Version 1 -> 2
- renumbered D104 to D2, SW102 to SW2, SW101 to SW3, U1 to U4
Connections:
- net SPI2_SDA1 is gone; now on net SPI2_CS0_DISP: U4.19 (IO11)
- net +3V3: now also R16.2; no longer R16.1
- net Chip Enable/Reset: now also R16.1; no longer R16.2
- net SPI2_CS0_DISP: no longer U4.22 (IO14)
- net SPI2_SDA0 renamed SPI2_SDA
- net SPI2_SDA2 renamed DISP_RS
- net SPI2_SDA3 renamed DISP_RESET
Other:
- moved on the sheet: R16

Commit message: Work in Progress of RTC Added Sheet Titles
Other:
- company: (none) -> Hochschule Luzern, Technik & Architektur
- title: (none) -> M.P.T MCU
Changed lines of the file:
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@@
 	(generator_version "10.0")
 	(paper "A4")
+	(title_block
+		(title "M.P.T MCU")
+		(company "Hochschule Luzern, Technik & Architektur")
+	)
 	(junction
 		(at 60.96 92.71)
