File: mpt_user_buttons.kicad_sch (KiCad schematic)
At the start: 0 parts

Commit message: Work in Progress of RTC Added Sheet Titles
Other:
- title: (none) -> M.P.T User Buttons
Changed lines of the file:
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@@
 	(paper "A4")
 	(title_block
+		(title "M.P.T User Buttons")
 		(company "Hochschule Luzern, Technik & Architektur")
 	)
